File: hardware/design/joystick-mouse.kicad_sch (KiCad schematic)
At the start: 9 parts

Commit message: unit tests
Parts:
- Joystick-Module1: renamed from Joystick-Module; footprint (none) -> COM-09032:XDCR_COM-09032
- back_sw1: renamed from back_sw; footprint (none) -> Button_Switch_THT:SW_XKB_DM1-16UP-1
- forward_sw1: renamed from forward_sw; footprint (none) -> Button_Switch_THT:SW_XKB_DM1-16UP-1
- left_sw1: renamed from left_sw; footprint (none) -> Button_Switch_THT:SW_XKB_DM1-16UP-1
- middle_sw1: renamed from middle_sw; footprint (none) -> Button_Switch_THT:SW_XKB_DM1-16UP-1
- mouse_wheel1: renamed from mouse_wheel; footprint (none) -> Rotary_Encoder:RotaryEncoder_Bourns_Horizontal_PEC12R-2x17F-Nxxxx
- right_sw1: renamed from right_sw; footprint (none) -> Button_Switch_THT:SW_XKB_DM1-16UP-1
- slider1: renamed from slider; footprint (none) -> Potentiometer_THT:Potentiometer_Bourns_PTA3043_Single_Slide
- renumbered Arduino_Nano to Arduino_Nano1
Other:
- moved on the sheet: Arduino_Nano1

Commit message: finish pcb
Parts:
- Joystick-Module1: footprint COM-09032:XDCR_COM-09032 -> ky-023_joystick:ky-023_joystick
Connections:
- net at slider1.2: now also Arduino_Nano1.26 (A7); no longer Arduino_Nano1.19 (A0)
- net at forward_sw1.2 (B): now also Arduino_Nano1.11 (D8); no longer Arduino_Nano1.9 (D6)
- net at Arduino_Nano1.25 (A6): now also Joystick-Module1.5 (SW)
- new net: Arduino_Nano1.9 (D6), middle_sw1.2 (B)
Other:
- moved on the sheet: forward_sw1, middle_sw1, slider1
